File: board-files/LEVER-board-production-0 (SENT to OSHPark).sch (EAGLE design)
At the start: 21 parts, among them Q3 MPSA42, U1 L78M

Commit message: opened in latest EAGLE sw
Parts:
- renumbered 1:12_TRNSFRMR to 1_12_TRNSFRMR
Changed lines of the file:
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@@
 <?xml version="1.0" encoding="utf-8"?>
 <!DOCTYPE eagle SYSTEM "eagle.dtd">
-<eagle version="6.6.0">
+<eagle version="7.5.0">
 <drawing>
 <settings>
@@
 </classes>
 <parts>
-<part name="1:12_TRNSFRMR" library="AKA_test" deviceset="PA0367" device=""/>
+<part name="1_12_TRNSFRMR" library="AKA_test" deviceset="PA0367" device=""/>
 <part name="D1" library="AKA_test" deviceset="QH03BZ600" device="" value="RB751"/>
 <part name="C1" library="adafruit" deviceset="C-US" device="C1812" value="2.2uF"/>
@@
 </plain>
 <instances>
-<instance part="1:12_TRNSFRMR" gate="G$1" x="5.08" y="121.92"/>
+<instance part="1_12_TRNSFRMR" gate="G$1" x="5.08" y="121.92"/>
 <instance part="D1" gate="D$1" x="53.34" y="139.7"/>
 <instance part="C1" gate="G$1" x="68.58" y="124.46"/>
@@
 <label x="45.72" y="104.14" size="1.778" layer="95"/>
 <label x="81.28" y="104.14" size="1.778" layer="95"/>
-<pinref part="1:12_TRNSFRMR" gate="G$1" pin="4"/>
+<pinref part="1_12_TRNSFRMR" gate="G$1" pin="4"/>
 <wire x1="10.16" y1="116.84" x2="27.94" y2="116.84" width="0.1524" layer="91"/>
 <wire x1="27.94" y1="116.84" x2="27.94" y2="104.14" width="0.1524" layer="91"/>
@@
 <net name="N$1" class="0">
 <segment>
-<pinref part="1:12_TRNSFRMR" gate="G$1" pin="3"/>
+<pinref part="1_12_TRNSFRMR" gate="G$1" pin="3"/>
 <wire x1="-15.24" y1="116.84" x2="-33.02" y2="116.84" width="0.1524" layer="91"/>
 <wire x1="-33.02" y1="116.84" x2="-33.02" y2="106.68" width="0.1524" layer="91"/>
@@
 <net name="N$3" class="0">
 <segment>
-<pinref part="1:12_TRNSFRMR" gate="G$1" pin="1"/>
+<pinref part="1_12_TRNSFRMR" gate="G$1" pin="1"/>
 <wire x1="10.16" y1="142.24" x2="30.48" y2="142.24" width="0.1524" layer="91"/>
 <wire x1="30.48" y1="142.24" x2="33.02" y2="139.7" width="0.1524" layer="91"/>
@@
 </segment>
 <segment>
-<pinref part="1:12_TRNSFRMR" gate="G$1" pin="2"/>
+<pinref part="1_12_TRNSFRMR" gate="G$1" pin="2"/>
 <wire x1="-15.24" y1="142.24" x2="-33.02" y2="142.24" width="0.1524" layer="91"/>
 <wire x1="-33.02" y1="142.24" x2="-33.02" y2="160.02" width="0.1524" layer="91"/>
